Commit message: interminent push

File: assets/newton/newton.urdf (robot description, URDF)
Before this commit: robot solo, 17 links, 16 joints
Links:
- link FL_SHOULDER: mass 0.14196048 -> 0.28196048
- link FL_UPPER_LEG: mass 0.14737324 -> 0.28737324
- link FR_SHOULDER: mass 0.14196048 -> 0.28196048
- link FR_UPPER_LEG: mass 0.14737324 -> 0.28737324
- link HL_SHOULDER: mass 0.14196048 -> 0.28196048
- link HL_UPPER_LEG: mass 0.14737324 -> 0.28737324
- link HR_SHOULDER: mass 0.14196048 -> 0.28196048
- link HR_UPPER_LEG: mass 0.14737324 -> 0.28737324
- link base_link: mass 1.25123725 -> 0.7
Joints:
- joint FL_HAA: type revolute -> fixed
- joint FR_HAA: type revolute -> fixed
- joint HL_HAA: type revolute -> fixed
- joint HR_HAA: type revolute -> fixed
